File: uq_phone/breakout_boards/display/display.kicad_pcb (KiCad board)
At the start: 2 copper layers, 26 x 34 mm, 8 parts, among them J1 541324562, J3 Conn_02x12_Odd_Even, U1 MCP1664T-E/OT

Commit message: Update display
Parts:
- added J2: 541324562, 541324562:CON_541324562_MOL, B.Cu at (74.5, 55.2)
Routing:
- net GND: track 8.74 -> 17.7 mm
- net +3.3V: track 64.1 -> 70.8 mm, vias 0 -> 1
- net DISP_DB3: track 23.9 -> 29.3 mm, vias 0 -> 1
- net DISP_DB2: track 22.0 -> 27.3 mm, vias 0 -> 1
- net DISP_DB1: track 20.1 -> 25.3 mm, vias 0 -> 1
- net DISP_DB0: track 18.6 -> 23.6 mm, vias 0 -> 1
- net DISP_WR: track 17.9 -> 22.8 mm, vias 0 -> 1
- net DISP_DC: track 17.1 -> 21.7 mm, vias 0 -> 1
- net DISP_CS: track 17.9 -> 22.3 mm, vias 0 -> 1
- net DISP_DB4: track 25.8 -> 30.1 mm, vias 0 -> 1
- net DISP_LEDK: track 16.4 -> 20.3 mm, vias 2 -> 3
- net DISP_DB12: track 17.3 -> 20.8 mm
- net DISP_DB9: track 16.5 -> 19.6 mm
- net DISP_DB5: track 27.7 -> 30.7 mm, vias 0 -> 1
- net DISP_DB11: track 16.1 -> 19.2 mm
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