File: uq_phone/breakout_boards/display/display.kicad_sch (KiCad schematic)
At the start: 8 parts, among them J1 541324562, J3 Conn_02x12_Odd_Even, U1 MCP1664T-E/OT

Commit message: Clean up and add DNP
Changed lines of the file:
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@@
 (kicad_sch
-	(version 20231120)
+	(version 20250114)
 	(generator "eeschema")
-	(generator_version "8.0")
+	(generator_version "9.0")
 	(paper "A4")
+	(text "Backlight Driver\n"
+		(exclude_from_sim no)
+		(at 87.884 27.178 0)
+		(effects
+			(font
+				(size 4 4)
+				(thickness 1)
+				(bold yes)
+			)
+		)
+	)
+	(text "CONFIRM FOOTPRINT PINS\n"
+		(exclude_from_sim no)
+		(at 180.086 33.02 0)
+		(effects
+			(font
+				(size 1.27 1.27)
+			)
+		)
+	)
+	(text "Display"
+		(exclude_from_sim no)
+		(at 209.296 19.812 0)
+		(effects
+			(font
+				(size 4 4)
+				(thickness 1)
+				(bold yes)
+			)
+		)
+	)
+	(text "Suits: \nAFR240320A0-2.0INTM"
+		(exclude_from_sim no)
+		(at 223.52 29.718 0)
+		(effects
+			(font
+				(size 1.27 1.27)
+			)
+		)
+	)
+	(text "Iout = 0.3/R\n3.83R -> 78mA"
+		(exclude_from_sim no)
+		(at 85.09 78.994 0)
+		(effects
+			(font
+				(size 1.27 1.27)
+			)
+		)
+	)
 	(junction
 		(at 204.47 132.08)
@@
 		)
 	)
-	(text "Backlight Driver\n"
-		(exclude_from_sim no)
-		(at 87.884 27.178 0)
-		(effects
-			(font
-				(size 4 4)
-				(thickness 1)
-				(bold yes)
-			)
-		)
-	)
-	(text "CONFIRM FOOTPRINT PINS\n"
-		(exclude_from_sim no)
-		(at 180.086 33.02 0)
-		(effects
-			(font
-				(size 1.27 1.27)
-			)
-		)
-	)
-	(text "Display"
-		(exclude_from_sim no)
-		(at 209.296 19.812 0)
-		(effects
-			(font
-				(size 4 4)
-				(thickness 1)
-				(bold yes)
-			)
-		)
-	)
-	(text "Suits: \nAFR240320A0-2.0INTM"
-		(exclude_from_sim no)
-		(at 223.52 29.718 0)
-		(effects
-			(font
-				(size 1.27 1.27)
-			)
-		)
-	)
-	(text "Iout = 0.3/R\n3.83R -> 78mA"
-		(exclude_from_sim no)
-		(at 85.09 78.994 0)
-		(effects
-			(font
-				(size 1.27 1.27)
-			)
-		)
-	)
 	(global_label "DISP_DB11"
 		(shape input)
@@
 		)
 	)
+	(embedded_fonts no)
 )
