File: uq_phone/power.kicad_sch (KiCad schematic)
At the start: 32 parts, among them J1 USB4105-GF-A, J2 S3B-PH-SM4-TB_LF__SN_, U1 MCP73871-2CCI_ML, U2 TPS62162DSGR, U3 BQ27441DRZR-G1A

Commit message: Update Various Connectors
Parts:
- removed J2: S3B-PH-SM4-TB_LF__SN_, S3B-PH-SM4-TB_LF__SN_:JST_S3B-PH-SM4-TB_LF__SN_, symbol S3B-PH-SM4-TB_LF__SN_:S3B-PH-SM4-TB_LF__SN_
- removed R3: 1k, Resistor_SMD:R_0402_1005Metric, symbol Resistors:Resistor_1k
- added B1: 113450, symbol Misc:Battery
- added J2: 0532610371, 0532610371:MOLEX_0532610371, symbol 0532610371:0532610371
- added R3: 2.2k, Resistor_SMD:R_0402_1005Metric, symbol Resistors:Resistor_2k2
Connections:
- net BAT_THERM: now also J2.3
- net GND: now also J2.2, R3.2
- net at U1.13 (PROG1): now also R3.1
- net at C6.1, R8.1, U3.6 (BAT)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: now also J2.1
Other:
- note added: "Charge Rate. =1000/RProg1 = 0.45A"
- note removed: "Charge Rate. =1000/RProg1 = 1A"
- moved on the sheet: C5, C6, R7, R8, R9, U3

Commit message: Generate Early production outputs
Parts:
- removed J2: 0532610371, 0532610371:MOLEX_0532610371, symbol 0532610371:0532610371
- added J2: BM03B-ACHSS-GAN-TF_LF__SN_, BM03B-ACHSS-GAN-TF_LF__SN_:JST_BM03B-ACHSS-GAN-TF_LF__SN_, symbol BM03B-ACHSS-GAN-TF_LF__SN_:BM03B-ACHSS-GAN-TF_LF__SN_
- B1: now not fitted
- C1, C4: LCSC PN (none) -> C2168196
- C2, C3: LCSC PN (none) -> C191541
- C5: LCSC PN (none) -> C26412
- C6: LCSC PN (none) -> C52923
- C7: LCSC PN (none) -> C3020456
- R1: LCSC PN (none) -> C131553
- R10: LCSC PN (none) -> C844811
- R11, R2, R4: LCSC PN (none) -> C606167
- R3: LCSC PN (none) -> C606171
- R5, R6, R9: LCSC PN (none) -> C7334585
- R7: LCSC PN (none) -> C851848
- R8: LCSC PN (none) -> PE0805FRE470R01Z
- U1: LCSC PN (none) -> C5121473
- U2: LCSC PN (none) -> C40256
- U3: LCSC PN (none) -> C473397
Connections:
- net BAT_THERM: now also J2.2
- net GND: now also J2.1
- net at C6.1, R8.1, U3.6 (BAT)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: now also J2.3

Commit message: Fix outputs
Parts:
- R8: LCSC PN PE0805FRE470R01Z -> C723359
Changed lines of the file:
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@@
 			)
 		)
-		(property "LCSC PN" "PE0805FRE470R01Z"
+		(property "LCSC PN" "C723359"
 			(at 233.68 233.68 0)
 			(effects
