File: uq_phone/breakout_boards/front_board/front_board.kicad_pcb (KiCad board)
At the start: 2 copper layers, 42.8 x 103.7 mm, 61 parts, among them J5 FI-RE51S-HF-R1500, J9 541324562, SW1 SKTAAAE010, SW10 SKTAAAE010, SW11 SKTAAAE010, SW12 SKTAAAE010, SW13 SKTAAAE010, SW14 SKTAAAE010, SW15 SKTAAAE010, SW16 SKTAAAE010, SW17 SKTAAAE010, SW18 SKTAAAE010, SW19 SKTAAAE010, SW2 SKTAAAE010, SW20 SKTAAAE010, SW21 SKTAAAE010, SW22 SKTAAAE010, SW23 SKTAAAE010, SW24 SKTAAAE010, SW25 SKTAAAE010, SW27 SKTAAAE010, SW29 SKTAAAE010, SW3 SKTAAAE010, SW31 SKTAAAE010, SW33 SKTAAAE010, SW34 SKTAAAE010, SW35 SKTAAAE010, SW36 SKTAAAE010, SW37 SKTAAAE010, SW38 SKTAAAE010, SW39 SKTAAAE010, SW4 SKTAAAE010, SW40 SKTAAAE010, SW41 SKTAAAE010, SW42 SKTAAAE010, SW43 SKSCLCE010, SW44 SKSCLCE010, SW45 SKSCLCE010, SW5 SKTAAAE010, SW6 SKTAAAE010, SW7 SKTAAAE010, SW8 SKTAAAE010, SW9 SKTAAAE010

Commit message: Update Various Connectors
Parts:
- removed J5: FI-RE51S-HF-R1500, FI-RE51S-HF-R1500:JAE_FI-RE51S-HF-R1500
- added J1: 6871XX14022_68715014022, 6871XX14022_68715014022:68715014022, B.Cu at (98.2, 105.2)
Routing:
- net PB_MENU_L: track 41.1 -> 43.2 mm
- net +3.3V: track 143.6 -> 144.7 mm
- net GND: vias 25 -> 60

Commit message: Fix outputs
Parts:
- removed R23: 0R, Resistor_SMD:R_0603_1608Metric
- added R1: 0R, Resistor_SMD:R_0603_1608Metric, F.Cu at (61.6, 104.6)
- moved SW44 1.91 mm to (99.5, 60.0)
- moved SW43 1.91 mm to (99.5, 71.5)
- moved SW45 1.91 mm to (99.5, 84.5)
- moved SW25 1.36 mm to (74.0, 112.6)
- moved SW19 1.36 mm to (68.2, 122.0)
- moved SW20 1.36 mm to (68.2, 126.0)
- moved SW21 1.36 mm to (80.2, 122.0)
- moved SW22 1.36 mm to (80.2, 126.0)
- moved SW23 1.36 mm to (92.2, 122.0)
- moved SW24 1.36 mm to (92.2, 126.0)
- moved SW27 1.36 mm to (80.2, 106.4)
- moved SW29 1.36 mm to (86.5, 112.6)
- moved SW31 1.36 mm to (80.2, 118.8)
- moved SW33 1.36 mm to (80.2, 110.6)
- moved SW34 1.36 mm to (80.2, 114.6)
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Routing:
- net +3.3V: track 144.7 -> 139.3 mm
- net PB_END_CALL: track 21.0 -> 20.1 mm
- net PB_DPAD_DOWN: track 19.4 -> 20.2 mm
- net GND: vias 60 -> 63
