File: uq_phone_v0.1.0/mcu.kicad_sch (KiCad schematic)
At the start: 22 parts, among them J6 Conn_ARM_SWD_TagConnect_TC2030, U5 TXB0108RGYR, U6 TXB0108RGYR, U7 STM32H733VGTx

Commit message: Clean repo
Connections:
- net +3.3V: now also U7.21 (VDDA), U7.6 (VBAT)
- no-connect marks 6 -> 4
