File: uq_phone_v0.1.0/uq_phone.kicad_pcb (KiCad board)
At the start: 4 copper layers, 42.8 x 103.8 mm, 146 parts, among them J1 USB4105-GF-A, J10 SJ-3551B-MSMT-TR-67, J11 Conn_01x02, J2 BM03B-ACHSS-GAN-TF_LF__SN_, J3 20279-001E-03, J4 20279-001E-03, J5 6871XX14022_68715014022, J6 Conn_ARM_SWD_TagConnect_TC2030, J7 Conn_01x02, J8 KP15B-6S-SF_800_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

Commit message: Clean repo
Connections:
- U7 pad 21: unconnected-(U7-VDDA-Pad21) -> +3.3V
- U7 pad 6: unconnected-(U7-VBAT-Pad6) -> +3.3V
Routing:
- net +3.3V: track 246.4 -> 262.4 mm
- net GND: track 81.8 -> 86.4 mm
