File: uq_phone_v0.2.0/uq_phone.kicad_pcb (KiCad board)
At the start: 6 copper layers, 111.8 x 108.6 mm, 205 parts, among them J1 PJ-242C, J10 513382474, J11 513382474, J2 124018312112A, J3 BM03B-ACHSS-GAN-TF_LF__SN_, J4 20279-001E-03, J5 20279-001E-03, J6 Conn_ARM_SWD_TagConnect_TC2030, J7 559092474, J8 MCS-302S-C1, J9 559092474, M1 C08-00A, Q1 MMBT3904LP-7, Q2 MMBT3904LP-7, Q3 S8050, SW1 SKTAAAE010, SW10 SKTAAAE010, SW11 SKTAAAE010, SW12 SKTAAAE010, SW13 SKTAAAE010, SW14 SKTAAAE010, SW15 SKTAAAE010, SW16 SKSCLCE010, SW17 SKTAAAE010, SW18 SKTAAAE010, SW19 SKTAAAE010, SW2 SKTAAAE010, SW20 SKTAAAE010, SW21 SKTAAAE010, SW22 SKSCLCE010, SW23 SKTAAAE010, SW24 SKTAAAE010, SW25 SKTAAAE010, SW26 SKTAAAE010, SW27 SKTAAAE010, SW28 SKTAAAE010, SW29 SKTAAAE010, SW3 SKTAAAE010, SW30 SKTAAAE010, SW31 SKTAAAE010, SW32 SKTAAAE010, SW33 SKTAAAE010, SW34 SKTAAAE010, SW35 SKTAAAE010, SW36 SKTAAAE010, SW37 SKTAAAE010, SW38 SKTAAAE010, SW39 SKTAAAE010, SW4 SKTAAAE010, SW40 SKTAAAE010, SW41 SKTAAAE010, SW5 SKTAAAE010, SW6 SKSCLCE010, SW7 SKTAAAE010, SW8 SKTAAAE010, SW9 SKTAAAE010, U1 TPS62162DSGR, U10 TPD8F003DQDR, U11 LSM6DSVTR, U12 DRV2603RUNR, U13 TS3A5018RSVR, U14 NAU88C22YG, U15 TPS22964CYZPR, U16 TXB0108YZPR2, U2 MCP73871-2CCI_ML, U3 BQ27441DRZR-G1A, U4 WP SNAP-IN BASE_6000636, U5 TCA9509MRVHR, U6 STM32H733VGHx, U7 TXB0108YZPR2, U8 TPD3F303DQDR

Commit message: More routing and placements
Parts:
- added LED18: XL-1010RGBC, custom_footprints:XL-1010RGBC-WS2812B, B.Cu at (40.8, 119.2)
- added LED20: XL-1010RGBC, custom_footprints:XL-1010RGBC-WS2812B, B.Cu at (40.8, 112.5)
- added LED21: XL-1010RGBC, custom_footprints:XL-1010RGBC-WS2812B, B.Cu at (53.0, 112.5)
- added LED22: XL-1010RGBC, custom_footprints:XL-1010RGBC-WS2812B, B.Cu at (28.5, 119.2)
- added LED23: XL-1010RGBC, custom_footprints:XL-1010RGBC-WS2812B, B.Cu at (40.8, 105.8)
- added LED24: XL-1010RGBC, custom_footprints:XL-1010RGBC-WS2812B, B.Cu at (53.0, 105.8)
- added LED25: XL-1010RGBC, custom_footprints:XL-1010RGBC-WS2812B, B.Cu at (28.5, 112.5)
- added LED26: XL-1010RGBC, custom_footprints:XL-1010RGBC-WS2812B, B.Cu at (40.8, 99.9)
- added LED27: XL-1010RGBC, custom_footprints:XL-1010RGBC-WS2812B, B.Cu at (53.0, 99.9)
- added LED28: XL-1010RGBC, custom_footprints:XL-1010RGBC-WS2812B, B.Cu at (28.5, 105.8)
- added LED31: XL-1010RGBC, custom_footprints:XL-1010RGBC-WS2812B, B.Cu at (28.5, 99.9)
- C36, C37, C48, C49, Q3, R21, R26, R27, R36, R38, R39, R40: moved to B.Cu
- MK1: moved to F.Cu
- moved TP1 64.2 mm to (40.8, 54.0)
- moved R21 49.5 mm to (60.4, 79.1), turned to 90 degrees
- moved R26 49.0 mm to (59.6, 79.1)
- moved Q3 46.8 mm to (59.1, 81.7), turned to 180 degrees
- moved R27 45.7 mm to (57.3, 80.6), turned to 180 degrees
- moved SW35 36.4 mm to (24.3, 118.4), turned to 90 degrees
- moved LED5 36.2 mm to (28.5, 116.9), turned to 180 degrees
- moved SW7 34.7 mm to (57.3, 112.5), turned to 90 degrees
- moved LED11 29.0 mm to (28.5, 103.5), turned to 180 degrees
- moved LED8 28.9 mm to (28.5, 110.2), turned to 180 degrees
- moved SW34 28.5 mm to (36.5, 117.9), turned to -90 degrees
- moved LED15 28.3 mm to (28.5, 85.1), turned to 180 degrees
- moved SW8 27.8 mm to (45.0, 112.5), turned to 90 degrees
- moved LED14 27.3 mm to (28.5, 96.7), turned to 180 degrees
- moved SW40 26.4 mm to (32.8, 118.4), turned to 90 degrees
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Connections:
- J10 pad 1: unconnected-(J10-Pad1) -> MOB_PWR
- J10 pad 10: unconnected-(J10-Pad10) -> MOB_AUD_IN
- J10 pad 11: unconnected-(J10-Pad11) -> MOB_AUD_OUT
- J10 pad 12: unconnected-(J10-Pad12) -> MOB_AUD_SYNC
- J10 pad 13: unconnected-(J10-Pad13) -> MOB_DCD
- J10 pad 14: unconnected-(J10-Pad14) -> MOB_DTR
- J10 pad 15: unconnected-(J10-Pad15) -> MOB_DSR
- J10 pad 16: unconnected-(J10-Pad16) -> MOB_TXD
- J10 pad 17: unconnected-(J10-Pad17) -> MOB_RTS
- J10 pad 18: unconnected-(J10-Pad18) -> MOB_CTS
- J10 pad 19: unconnected-(J10-Pad19) -> MOB_RXD
- J10 pad 2: unconnected-(J10-Pad2) -> MOB_RST
- J10 pad 20: unconnected-(J10-Pad20) -> MOB_RI
- J10 pad 21: unconnected-(J10-Pad21) -> SIM_RST
- J10 pad 22: unconnected-(J10-Pad22) -> SIM_CLK
- J10 pad 23: GND -> SIM_DATA
- J10 pad 24: GND -> SIM_VDD
- J10 pad 3: unconnected-(J10-Pad3) -> MOB_SAFE_PWR_REMOVE_L
- J10 pad 4: unconnected-(J10-Pad4) -> MOB_WAKE_L
- J10 pad 9: unconnected-(J10-Pad9) -> MOB_AUD_BCLK
- J9 pad 1: unconnected-(J9-Pad1) -> MOB_PWR
- J9 pad 10: unconnected-(J9-Pad10) -> MOB_AUD_IN
- J9 pad 11: unconnected-(J9-Pad11) -> MOB_AUD_OUT
- J9 pad 12: unconnected-(J9-Pad12) -> MOB_AUD_SYNC
- J9 pad 13: unconnected-(J9-Pad13) -> MOB_DCD
- J9 pad 14: unconnected-(J9-Pad14) -> MOB_DTR
- J9 pad 15: unconnected-(J9-Pad15) -> MOB_DSR
- J9 pad 16: unconnected-(J9-Pad16) -> MOB_TXD
- J9 pad 17: unconnected-(J9-Pad17) -> MOB_RTS
- J9 pad 18: unconnected-(J9-Pad18) -> MOB_CTS
- J9 pad 19: unconnected-(J9-Pad19) -> MOB_RXD
- J9 pad 2: unconnected-(J9-Pad2) -> MOB_RST
- J9 pad 20: unconnected-(J9-Pad20) -> MOB_RI
- J9 pad 3: unconnected-(J9-Pad3) -> MOB_SAFE_PWR_REMOVE_L
- J9 pad 4: unconnected-(J9-Pad4) -> MOB_WAKE_L
- J9 pad 9: unconnected-(J9-Pad9) -> MOB_AUD_BCLK
- U4 pad 152: MOB_SAFE_PWR_REMOVE -> MOB_SAFE_PWR_REMOVE_L
- U4 pad 22: MOB_SYS_CLK -> unconnected-(U4A-SYS_CLK-Pad22)
- U6 pad A1: PB_6 -> MOB_RST_CTL
- U6 pad A2: PB_5 -> MOB_PWR_CTL
- U6 pad G5: MOB_PWR_CTL -> unconnected-(U6-PB2-PadG5)
- U6 pad H4: HP_DET_MCU -> unconnected-(U6-PC5-PadH4)
- U6 pad J10: unconnected-(U6-PD13-PadJ10) -> HP_DET_MCU
- U6 pad J4: AUD_SW_H -> unconnected-(U6-PB0-PadJ4)
- U6 pad J9: unconnected-(U6-PD9-PadJ9) -> MOB_SAFE_PWR_REMOVE_H
- U6 pad K10: unconnected-(U6-PD12-PadK10) -> AUD_SW_H
- U6 pad K4: MOB_WAKE_H -> unconnected-(U6-PB1-PadK4)
- U6 pad K7: MOB_RST_CTL -> PB_5
- U6 pad K8: unconnected-(U6-PB12-PadK8) -> PB_6
- U6 pad K9: unconnected-(U6-PD8-PadK9) -> MOB_WAKE_H
- U7 pad A1: unconnected-(U7-B2-PadA1) -> MOB_SAFE_PWR_REMOVE_H
- U7 pad A4: unconnected-(U7-A2-PadA4) -> MOB_SAFE_PWR_REMOVE_L
Routing:
- net LED_DATA: track 0.00 -> 89.8 mm, vias 1 -> 2
- net MOB_WAKE_L: track 2.53 -> 45.9 mm, vias 1 -> 2
- net SWDIO: track 0.00 -> 42.9 mm, vias 1 -> 3
- net RST: track 0.00 -> 41.8 mm, vias 1 -> 2
- net SWCLK: track 0.00 -> 40.1 mm, vias 1 -> 3
- net MOB_SAFE_PWR_REMOVE_L: track 0.00 -> 38.4 mm, vias 0 -> 2
- net AUD_SDA: track 0.00 -> 38.2 mm, vias 0 -> 2
- net SWO: track 0.00 -> 38.0 mm, vias 1 -> 3
- net AUD_SCL: track 0.00 -> 36.5 mm, vias 0 -> 2
- net MOB_AUD_IN: track 4.23 -> 28.4 mm, vias 1 -> 4
- net MOB_AUD_OUT: track 3.36 -> 26.9 mm, vias 1 -> 4
- net MOB_AUD_SYNC: track 5.40 -> 28.8 mm, vias 1 -> 4
- net MOB_AUD_BCLK: track 6.01 -> 29.0 mm, vias 1 -> 4
- net SPEAKER_N: track 0.00 -> 18.5 mm, vias 0 -> 2
- net SPEAKER_P: track 0.00 -> 17.8 mm, vias 0 -> 2
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Other:
- outline, holes or cut-outs redrawn

Commit message: Another day of routing and adding components
Parts:
- removed C36: 4.7uF, Capacitor_SMD:C_0201_0603Metric
- removed C37, C48, C49: 1uF, Capacitor_SMD:C_0201_0603Metric
- removed J1: PJ-242C, custom_footprints:PJ-242C
- removed LED2: XL-1010RGBC, custom_footprints:XL-1010RGBC-WS2812B
- removed R36: 2.2k, Resistor_SMD:R_0201_0603Metric
- removed R38: 47k, Resistor_SMD:R_0201_0603Metric
- removed R39, R40: 10k, Resistor_SMD:R_0201_0603Metric
- added C27: 220uF, Capacitor_SMD:C_1206_3216Metric, F.Cu at (87.5, 33.0)
- added C52: 220uF, Capacitor_SMD:C_1206_3216Metric, F.Cu at (87.5, 30.6)
- added C53: 220uF, Capacitor_SMD:C_1206_3216Metric, F.Cu at (87.5, 28.4)
- added D10: ESD5451X, custom_footprints:WBFBP-02C_L1.0-W0.6-BI, F.Cu at (67.0, 121.1)
- added D11: ESD5451X, custom_footprints:WBFBP-02C_L1.0-W0.6-BI, F.Cu at (67.0, 122.9)
- added D12: ESD5451X, custom_footprints:WBFBP-02C_L1.0-W0.6-BI, F.Cu at (67.0, 124.7)
- added D8: ESD5451X, custom_footprints:WBFBP-02C_L1.0-W0.6-BI, F.Cu at (67.0, 117.5)
- added D9: ESD5451X, custom_footprints:WBFBP-02C_L1.0-W0.6-BI, F.Cu at (67.0, 119.3)
- added LED19: XL-1010RGBC, custom_footprints:XL-1010RGBC-Alt, B.Cu at (53.1, 117.7)
- added U?: PJ-342C, custom_footprints:PJ-342C, F.Cu at (53.0, 121.2)
- C13: value 47uF -> 220uF; footprint Capacitor_SMD:C_0805_2012Metric -> Capacitor_SMD:C_1206_3216Metric
- MK1: moved to B.Cu
- moved R14 30.5 mm to (117.8, 40.1), turned to 0 degrees
- moved R12 30.1 mm to (117.8, 41.0), turned to 0 degrees
- moved R15 29.7 mm to (117.8, 42.0), turned to 0 degrees
- moved R13 29.5 mm to (117.8, 42.9), turned to 0 degrees
- moved TP9 13.8 mm to (107.0, 23.1)
- moved TP17 7.15 mm to (88.5, 25.7)
- moved TP8 7.15 mm to (88.5, 23.1)
- moved R42 6.23 mm to (28.6, 80.5), turned to 0 degrees
- moved TP4 4.53 mm to (88.4, 48.3)
- moved C9 3.91 mm to (88.6, 39.0)
- moved C8 3.91 mm to (88.6, 39.9)
- moved C13 2.24 mm to (87.5, 35.3)
- moved C12 1.96 mm to (88.1, 37.5)
- moved FB2 1.96 mm to (33.6, 25.9), turned to 90 degrees
- moved TP7 1.41 mm to (25.1, 29.3)
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Connections:
- U14 pad 15: HP_DET -> unconnected-(U14-CSB/GPIO1-Pad15)
Routing:
- net +3.3V: track 14.5 -> 152.8 mm, vias 9 -> 16
- net SCL: track 11.8 -> 123.7 mm, vias 4 -> 5
- net SDA: track 11.6 -> 122.8 mm, vias 4 -> 5
- net HP_RIGHT: track 0.00 -> 104.3 mm
- net HP_LEFT: track 0.00 -> 103.5 mm
- net MIC_BIAS: track 1.27 -> 103.6 mm, vias 0 -> 1
- net MIC_OUT: track 0.00 -> 101.6 mm, vias 0 -> 1
- net MIC_GND: track 0.00 -> 101.6 mm, vias 0 -> 1
- net Net-(U14-RMICN): track 1.12 -> 101.8 mm, vias 0 -> 1
- net HP_MIC: track 0.00 -> 100.3 mm, vias 0 -> 1
- net MOB_SAFE_PWR_REMOVE_L: track 38.4 -> 78.4 mm, vias 2 -> 4
- net MOB_PWR: track 9.41 -> 47.2 mm, vias 2 -> 4
- net +1.8V: track 9.97 -> 47.0 mm, vias 1 -> 6
- net MOB_AUD_BCLK: track 29.0 -> 64.4 mm, vias 4 -> 6
- net MOB_AUD_IN: track 28.4 -> 62.0 mm, vias 4 -> 6
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- added copper zone on B.Cu, net +1.8V
- added copper zone on B.Cu, net AGND
- added copper zone on F.Cu, net AGND
- added copper zone on In1.Cu, net AGND
- added copper zone on In2.Cu, net AGND
- added copper zone on In3.Cu, net AGND
- added copper zone on In4.Cu, net AGND
- added copper zone on B.Cu, net VBAT
- removed copper zone on In3.Cu, net GND
- removed copper zone on In4.Cu, net GND
Other:
- outline, holes or cut-outs redrawn

Commit message: More routing and moving cellular to new project
Parts:
- removed the REF** at (40.8, 84.3)
- removed U?: PJ-342C, custom_footprints:PJ-342C
- added C28: 100nF, Capacitor_SMD:C_0201_0603Metric, F.Cu at (69.3, 116.7)
- added C36: 4.7uF, Capacitor_SMD:C_0201_0603Metric, F.Cu at (69.3, 118.4)
- added C37: 1uF, Capacitor_SMD:C_0201_0603Metric, F.Cu at (69.3, 120.2)
- added C48: 1uF, Capacitor_SMD:C_0201_0603Metric, F.Cu at (69.3, 121.9)
- added C49: 1uF, Capacitor_SMD:C_0201_0603Metric, F.Cu at (69.3, 123.7)
- added LED2: XL-1010RGBC, custom_footprints:XL-1010RGBC-WS2812B, F.Cu at (14.8, 91.5)
- added R28: 100k, Resistor_SMD:R_0201_0603Metric, F.Cu at (71.7, 116.7)
- added R29: 10k, Resistor_SMD:R_0201_0603Metric, F.Cu at (71.7, 118.4)
- added R30: 10k, Resistor_SMD:R_0201_0603Metric, F.Cu at (71.7, 120.2)
- added R31: 47k, Resistor_SMD:R_0201_0603Metric, F.Cu at (71.7, 121.9)
- added R36: 2.2k, Resistor_SMD:R_0201_0603Metric, F.Cu at (71.7, 123.7)
- added REF**: CUI_SJ-43504-SMT-TR, SJ-43504-SMT-TR:CUI_SJ-43504-SMT-TR, B.Cu at (57.3, 125.6)
- moved MK1 7.25 mm to (64.9, 121.7)
- moved R42 6.61 mm to (21.9, 80.2), turned to 90 degrees
- moved TP5 3.19 mm to (28.9, 42.6)
- moved TP2 2.58 mm to (32.8, 41.0)
- moved D10 1.07 mm to (67.2, 120.0)
- moved D11 1.07 mm to (67.2, 121.8)
- moved D8 1.07 mm to (67.2, 116.5)
- moved D9 1.07 mm to (67.2, 118.2)
- moved D12 1.07 mm to (67.2, 123.7)
- moved LED26 0.75 mm to (40.8, 99.1)
- moved LED27 0.75 mm to (53.0, 99.1)
- moved LED31 0.75 mm to (28.5, 99.1)
- moved SW24 0.75 mm to (57.3, 99.1)
- moved SW25 0.75 mm to (36.5, 99.1)
- moved SW26 0.75 mm to (24.3, 99.1)
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Connections:
- U6 pad A3: PB_HASH -> unconnected-(U6-PE2-PadA3)
- U6 pad A5: PB_DPAD_SELECT -> unconnected-(U6-PB7-PadA5)
- U6 pad A6: PB_DPAD_DOWN -> unconnected-(U6-PB4(NJTRST)-PadA6)
- U6 pad A8: PB_END_CALL -> unconnected-(U6-PA15(JTDI)-PadA8)
- U6 pad B1: PB_7 -> PB_CALL
- U6 pad B3: PB_1 -> PB_DPAD_DOWN
- U6 pad B5: PB_DPAD_LEFT -> unconnected-(U6-PB6-PadB5)
- U6 pad B6: PB_DPAD_UP -> unconnected-(U6-PD5-PadB6)
- U6 pad C1: PB_8 -> PB_4
- U6 pad C3: PB_2 -> PB_1
- U6 pad C4: PB_0 -> unconnected-(U6-PE1-PadC4)
- U6 pad C5: PB_DPAD_RIGHT -> unconnected-(U6-PB5-PadC5)
- U6 pad C6: PB_CALL -> unconnected-(U6-PD6-PadC6)
- U6 pad D1: PB_9 -> unconnected-(U6-PH1-PadD1)
- U6 pad D3: PB_3 -> PB_7
- U6 pad D4: PB_STAR -> unconnected-(U6-PE0-PadD4)
- U6 pad E3: PB_4 -> PB_STAR
- U6 pad F1: PB_MENU_L -> PB_DPAD_SELECT
- U6 pad F2: PB_MENU_R -> PB_DPAD_UP
- U6 pad G2: PB_PWR -> PB_MENU_L
- U6 pad G4: VIB_EN -> PB_DPAD_LEFT
- U6 pad G7: unconnected-(U6-PE14-PadG7) -> DISP_SDA
- U6 pad G8: unconnected-(U6-PD15-PadG8) -> DISP_RESET
- U6 pad H8: unconnected-(U6-PD14-PadH8) -> DISP_DC
- U6 pad J3: VIB_PWM -> DISP_BL
- U6 pad J6: unconnected-(U6-PE12-PadJ6) -> DISP_SCL
- U6 pad J7: DISP_BL -> unconnected-(U6-PB10-PadJ7)
- U6 pad J8: unconnected-(U6-PB13-PadJ8) -> DISP_CS
- U6 pad K4: unconnected-(U6-PB1-PadK4) -> VIB_PWM
- U6 pad K5: unconnected-(U6-PE9-PadK5) -> VIB_EN
- U6 pad K7: PB_5 -> unconnected-(U6-PB11-PadK7)
- U6 pad K8: PB_6 -> unconnected-(U6-PB12-PadK8)
Routing:
- net +3.3V_SW: track 1.33 -> 296.3 mm, vias 0 -> 26
- net VIB_PWM: track 1.55 -> 136.6 mm
- net VIB_EN: track 0.82 -> 133.3 mm
- net PB_7: track 0.00 -> 107.7 mm, vias 1 -> 2
- net PB_4: track 0.00 -> 98.0 mm, vias 0 -> 2
- net PB_1: track 0.00 -> 92.0 mm, vias 1 -> 2
- net PB_DPAD_SELECT: track 0.00 -> 91.2 mm, vias 1 -> 2
- net PB_STAR: track 0.00 -> 91.1 mm
- net PB_DPAD_DOWN: track 0.00 -> 85.6 mm, vias 1 -> 2
- net PB_CALL: track 0.00 -> 79.6 mm, vias 1 -> 2
- net PB_DPAD_LEFT: track 0.00 -> 79.4 mm, vias 1 -> 2
- net PB_DPAD_UP: track 0.00 -> 79.0 mm, vias 1 -> 2
- net PB_MENU_L: track 0.00 -> 78.5 mm, vias 1 -> 2
- net +3.3V: track 152.8 -> 220.1 mm, vias 16 -> 25
- net DISP_BL: track 0.00 -> 63.1 mm, vias 1 -> 3
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- added copper zone on In1.Cu, net +3.3V
Other:
- outline, holes or cut-outs redrawn

Commit message: Most routing complete
Connections:
- U6 pad A3: unconnected-(U6-PE2-PadA3) -> PB_0
- U6 pad A5: unconnected-(U6-PB7-PadA5) -> PB_2
- U6 pad A6: unconnected-(U6-PB4(NJTRST)-PadA6) -> PB_3
- U6 pad B5: unconnected-(U6-PB6-PadB5) -> PB_9
- U6 pad B6: unconnected-(U6-PD5-PadB6) -> PB_6
- U6 pad C4: unconnected-(U6-PE1-PadC4) -> PB_8
- U6 pad C5: unconnected-(U6-PB5-PadC5) -> PB_5
- U6 pad C6: unconnected-(U6-PD6-PadC6) -> PB_DPAD_RIGHT
- U6 pad D4: unconnected-(U6-PE0-PadD4) -> PB_HASH
- U6 pad D6: unconnected-(U6-PD7-PadD6) -> PB_END_CALL
- U6 pad D7: unconnected-(U6-PD4-PadD7) -> PB_MENU_R
- U6 pad K8: unconnected-(U6-PB12-PadK8) -> PB_PWR
Routing:
- net PB_HASH: track 11.8 -> 125.2 mm, vias 1 -> 2
- net PB_9: track 11.7 -> 119.3 mm, vias 1 -> 2
- net PB_8: track 11.7 -> 113.0 mm, vias 1 -> 2
- net PB_6: track 11.7 -> 112.9 mm, vias 0 -> 2
- net PB_0: track 11.7 -> 112.7 mm, vias 1 -> 2
- net PB_5: track 11.7 -> 106.4 mm, vias 0 -> 2
- net PB_3: track 11.7 -> 104.7 mm, vias 1 -> 2
- net PB_2: track 11.7 -> 97.9 mm, vias 1 -> 2
- net PB_END_CALL: track 9.30 -> 89.5 mm, vias 1 -> 2
- net PB_MENU_R: track 9.30 -> 83.8 mm, vias 1 -> 2
- net PB_DPAD_RIGHT: track 0.75 -> 73.5 mm, vias 0 -> 2
- net unconnected-(U6-PE0-PadD4): track 8.23 -> 0.00 mm, vias 1 -> 0
- net unconnected-(U6-PD5-PadB6): track 5.94 -> 0.00 mm, vias 1 -> 0
- net unconnected-(U6-PB6-PadB5): track 5.85 -> 0.00 mm, vias 1 -> 0
- net unconnected-(U6-PB5-PadC5): track 5.64 -> 0.00 mm, vias 1 -> 0
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