File: uq_phone_v0.2.0/user_io.kicad_sch (KiCad schematic)
At the start: 29 parts, among them J5 6871XX14022_68715014022, J7 Conn_01x02, J8 KP15B-6S-SF_800_, J9 541324562, M1 VCDM0834B004L, U10 TPD3F303DQDR, U11 TPD8F003DQDR, U12 MCP1664T-E/OT, U8 LSM6DSVTR, U9 DRV2603RUNR

Commit message: Clean repo
Parts:
- removed Cable1: 0151660555, symbol Misc:Cable
- removed J5: 6871XX14022_68715014022, 6871XX14022_68715014022:68715014022, symbol 6871XX14022_68715014022:6871XX14022_68715014022
- removed J8: KP15B-6S-SF_800_, KP15B-6S-SF_800_:HIROSE_KP15B-6S-SF_800_, symbol KP15B-6S-SF_800_:KP15B-6S-SF_800_
- removed R28, R29: 0R, Resistor_SMD:R_0603_1608Metric, symbol Resistors:Resistor_0R
- added J8: MCS-302S-C1, custom_footprints:SIM-SMD_MCS-302S-C1, symbol Misc:MCS-302S-C1
- J9: now in the parts list
- renumbered C34 to C27, C35 to C28, C28 to C34, C27 to C35, J7 to J10, R33 to R25, R30 to R26, R31 to R27, R32 to R28, R34 to R29, U11 to U10, U8 to U11, U9 to U12, U10 to U8, U12 to U9
Connections:
- net +3.3V: now also J8.4 (VDD); no longer R25.2
- net GND: now also U12.3 (LRA/~{ERM}), J8.12 (SIM_1_GND), J8.6 (VSS)
- net SIM_VDD: now also J8.9 (SIM_1_VCC)
- net uSD_DET: no longer R25.1
- net at U10.16 (CH1_OUT): now also J8.1 (DAT2)
- net at U10.15 (CH2_OUT): now also J8.2 (CD/DAT3)
- net at U10.14 (CH3_OUT): now also J8.3 (CMD)
- net at U10.13 (CH4_OUT): now also J8.5 (CLK)
- net at U10.11 (CH6_OUT): now also J8.7 (DAT0)
- net at U10.10 (CH7_OUT): now also J8.8 (DAT1)
- net at U8.1 (DATA1_OUT): now also J8.10 (SIM_1_RST)
- net at U8.2 (CLK_OUT): now also J8.11 (SIM_1_CLK)
- net at U8.3 (DATA2_OUT): now also J8.14 (SIM_1_DATA)
- no-connect marks 14 -> 13
Other:
- note added: "TODO: Figure switch out"
- note added: "TODO: replace with footprint"
- note removed: "CONFIRM FOOTPRINT PINS"
- note removed: "Conn 50x"
- note removed: "Need to check STM pullups sufficient"
- moved on the sheet: R25, U10

Commit message: Add more footprints, reduce sizes
Parts:
- removed C29, C30, C31: 22pF, Capacitor_SMD:C_0402_1005Metric, symbol Capacitors:Capacitor_22pF
- removed J10: Conn_01x02, Connector_Wire:SolderWire-0.1sqmm_1x02_P3.6mm_D0.4mm_OD1mm, symbol Connector_Generic:Conn_01x02
- removed J9: 541324562, 541324562:CON_541324562_MOL, symbol 541324562:541324562
- removed M1: VCDM0834B004L, custom_footprints:Motor_8mm, symbol Misc:VCDM0834B004L
- removed R26, R27, R28: 22R, Resistor_SMD:R_0402_1005Metric, symbol Resistors:Resistor_22R
- added C29: 100nF, Capacitor_SMD:C_0201_0603Metric, symbol Capacitors:capacitor_100nF
- added Disp1: AFR240320A0-2.0INTM, custom_footprints:Display, symbol Misc:Display
- added M1: C08-00A, custom_footprints:Motor_8mm, symbol Misc:C08-00A
- C28: footprint Capacitor_SMD:C_0402_1005Metric -> Capacitor_SMD:C_0201_0603Metric; LCSC PN C191541 -> C335103
- C32, C34, C35: footprint Capacitor_SMD:C_0402_1005Metric -> Capacitor_SMD:C_0201_0603Metric; LCSC PN C307331 -> C160831
- R25: footprint Resistor_SMD:R_0402_1005Metric -> Resistor_SMD:R_0201_0603Metric; LCSC PN C851848 -> C106225
- R29: footprint Resistor_SMD:R_0603_1608Metric -> Resistor_SMD:R_0402_1005Metric; LCSC PN C3037044 -> C3013169
- U12: DESCRIPTION IC LRA/ERM HAPTIC DRIVER 10QFN -> (none)
Connections:
- net +3.3V: now also R25.2, U12.3 (LRA/~{ERM}), C29.1
- net GND: now also J8.22 (S/GND), J8.23 (GND), C29.2; no longer U12.3 (LRA/~{ERM})
- net SIM_CLK: now also U8.7 (CLK_IN)
- net SIM_DATA: now also U8.6 (DATA2_IN)
- net SIM_RST: now also U8.8 (DATA1_IN)
- net at U12.6 (OUT_M): now also M1.2 (-)
- net at U12.9 (OUT_P): now also M1.1 (+)
- net uSD_SIM_CD: now reaches R25.1
- net uSD_SIM_CD: now also J8.21 (SW/CD)
Other:
- note added: "TODO: Confirm Switch"
- note removed: "Suits: AFR240320A0-2.0INTM"
- note removed: "TODO: Figure switch out"
- moved on the sheet: C32, C33, J8A, J8B, R25, U10, U8

Commit message: Various Changes to footprints and components
Parts:
- removed L2: 4.7uH, WE-MAPI_3015:WE-MAPI_3015, symbol WE-MAPI_3015:WE-MAPI_3015
- added L2: 4.7uH, custom_footprints:IND-SMD_L2.0-W1.2_MTQH201208S4R7MBT, symbol Misc:MTQH201208S4R7MBT
Connections:
- net +3.3V: no longer C27.1, U9.5 (VIN)
- net at D2.2 (A), U9.1 (SW): now also L2.2
- new net +3.3V_SW: C27.1, L2.1, U9.5 (VIN)
Other:
- note removed: "TODO: replace with footprint"
- title: Power System -> UQ Phone
Changed lines of the file:
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@@
 	(paper "A3")
 	(title_block
-		(title "Power System")
+		(title "UQ Phone")
+		(rev "0.2.0")
 		(company "The University of Queensland")
 	)
@@
 		)
 	)
-	(text "TODO: replace with footprint\n"
-		(exclude_from_sim no)
-		(at 359.156 253.238 0)
-		(effects
-			(font
-				(size 1.27 1.27)
-			)
-		)
-	)
 	(text "Micro SIM card"
 		(exclude_from_sim no)
@@
 	(wire
 		(pts
+			(xy 350.52 41.91) (xy 340.36 41.91)
+		)
+		(stroke
+			(width 0)
+			(type default)
+		)
+	)
+	(wire
+		(pts
 			(xy 29.21 185.42) (xy 52.07 185.42)
 		)
@@
 	(wire
 		(pts
+			(xy 360.68 41.91) (xy 370.84 41.91)
+		)
+		(stroke
+			(width 0)
+			(type default)
+		)
+	)
+	(wire
+		(pts
 			(xy 313.69 123.19) (xy 312.42 123.19)
 		)
@@
 	(wire
 		(pts
-			(xy 351.79 41.91) (xy 340.36 41.91)
-		)
-		(stroke
-			(width 0)
-			(type default)
-		)
-	)
-	(wire
-		(pts
 			(xy 90.17 256.54) (xy 91.44 256.54)
 		)
@@
 	(wire
 		(pts
-			(xy 359.41 41.91) (xy 370.84 41.91)
-		)
-		(stroke
-			(width 0)
-			(type default)
-		)
-	)
-	(wire
-		(pts
 			(xy 50.8 187.96) (xy 50.8 190.5)
 		)
@@
 	(wire
 		(pts
+			(xy 91.44 227.33) (xy 91.44 229.87)
+		)
+		(stroke
+			(width 0)
+			(type default)
+		)
+	)
+	(wire
+		(pts
 			(xy 312.42 120.65) (xy 307.34 120.65)
 		)
@@
 	)
 	(symbol
-		(lib_id "WE-MAPI_3015:WE-MAPI_3015")
-		(at 355.6 41.91 0)
-		(unit 1)
-		(exclude_from_sim no)
-		(in_bom yes)
-		(on_board yes)
-		(dnp no)
-		(fields_autoplaced yes)
-		(property "Reference" "L2"
-			(at 355.6 35.56 0)
-			(effects
-				(font
-					(size 1.27 1.27)
-				)
-			)
-		)
-		(property "Value" "4.7uH"
-			(at 355.6 38.1 0)
-			(effects
-				(font
-					(size 1.27 1.27)
-				)
-			)
-		)
-		(property "Footprint" "WE-MAPI_3015:WE-MAPI_3015"
-			(at 355.6 41.91 0)
-			(effects
-				(font
-					(size 1.27 1.27)
-				)
-				(justify bottom)
-				(hide yes)
-			)
-		)
-		(property "Datasheet" ""
-			(at 355.6 41.91 0)
-			(effects
-				(font
-					(size 1.27 1.27)
-				)
-				(hide yes)
-			)
-		)
-		(property "Description" ""
-			(at 355.6 41.91 0)
-			(effects
-				(font
-					(size 1.27 1.27)
-				)
-				(hide yes)
-			)
-		)
-		(property "DigiKey_Part_Number" "732-4866-2-ND"
-			(at 355.6 41.91 0)
-			(effects
-				(font
-					(size 1.27 1.27)
-				)
-				(justify bottom)
-				(hide yes)
-			)
-		)
-		(property "SnapEDA_Link" "https://www.snapeda.com/parts/74438335047/W%25C3%25BCrth+Elektronik+Midcom/view-part/?ref=snap"
-			(at 355.6 41.91 0)
-			(effects
-				(font
-					(size 1.27 1.27)
-				)
-				(justify bottom)
-				(hide yes)
-			)
-		)
-		(property "Description_1" "\n                        \n                            Inductor SMD WE-MAPI Metal Alloy | Wurth Electronics 74438335047\n                        \n"
-			(at 355.6 41.91 0)
-			(effects
-				(font
-					(size 1.27 1.27)
-				)
-				(justify bottom)
-				(hide yes)
-			)
-		)
-		(property "MF" "Würth Elektronik"
-			(at 355.6 41.91 0)
-			(effects
-				(font
-					(size 1.27 1.27)
-				)
-				(justify bottom)
-				(hide yes)
-			)
-		)
-		(property "Package" "1212 Würth Elektronik"
-			(at 355.6 41.91 0)
-			(effects
-				(font
-					(size 1.27 1.27)
-				)
-				(justify bottom)
-				(hide yes)
-			)
-		)
-		(property "Check_prices" "https://www.snapeda.com/parts/74438335047/W%25C3%25BCrth+Elektronik+Midcom/view-part/?ref=eda"
-			(at 355.6 41.91 0)
-			(effects
-				(font
-					(size 1.27 1.27)
-				)
-				(justify bottom)
-				(hide yes)
-			)
-		)
-		(property "MP" "74438335047"
-			(at 355.6 41.91 0)
-			(effects
-				(font
-					(size 1.27 1.27)
-				)
-				(justify bottom)
-				(hide yes)
-			)
-		)
-		(property "LCSC PN" "C2761891"
-			(at 355.6 41.91 0)
-			(effects
-				(font
-					(size 1.27 1.27)
-				)
-				(hide yes)
-			)
-		)
-		(pin "2"
-		)
-		(pin "1"
-		)
-		(instances
-			(project ""
-				(path "/14f57415-6807-40a5-bb38-3cb818a2cdae/3e1644a6-29e0-4613-bdce-8513434c26aa"
-					(reference "L2")
-					(unit 1)
-				)
-			)
-		)
-	)
-	(symbol
 		(lib_id "Capacitors:capacitor_100nF")
 		(at 92.71 165.1 0)
@@
 	(symbol
 		(lib_id "power:+3.3V")
-		(at 91.44 229.87 0)
+		(at 91.44 227.33 0)
 		(unit 1)
 		(exclude_from_sim no)
@@
 		(fields_autoplaced yes)
 		(property "Reference" "#PWR094"
-			(at 91.44 233.68 0)
+			(at 91.44 231.14 0)
 			(effects
 				(font
@@
 		)
 		(property "Value" "+3.3V"
-			(at 91.44 224.79 0)
+			(at 91.44 222.25 0)
 			(effects
 				(font
@@
 		)
 		(property "Footprint" ""
-			(at 91.44 229.87 0)
+			(at 91.44 227.33 0)
 			(effects
 				(font
@@
 		)
 		(property "Datasheet" ""
-			(at 91.44 229.87 0)
+			(at 91.44 227.33 0)
 			(effects
 				(font
@@
 		)
 		(property "Description" "Power symbol creates a global label with name \"+3.3V\""
-			(at 91.44 229.87 0)
+			(at 91.44 227.33 0)
 			(effects
 				(font
@@
 	)
 	(symbol
+		(lib_id "power:+3.3V")
+		(at 325.12 52.07 0)
+		(unit 1)
+		(exclude_from_sim no)
+		(in_bom yes)
+		(on_board yes)
+		(dnp no)
+		(fields_autoplaced yes)
+		(property "Reference" "#PWR0208"
+			(at 325.12 55.88 0)
+			(effects
+				(font
+					(size 1.27 1.27)
+				)
+				(hide yes)
+			)
+		)
+		(property "Value" "+3.3V_SW"
+			(at 325.12 46.99 0)
+			(effects
+				(font
+					(size 1.27 1.27)
+				)
+			)
+		)
+		(property "Footprint" ""
+			(at 325.12 52.07 0)
+			(effects
+				(font
+					(size 1.27 1.27)
+				)
+				(hide yes)
+			)
+		)
+		(property "Datasheet" ""
+			(at 325.12 52.07 0)
+			(effects
+				(font
+					(size 1.27 1.27)
+				)
+				(hide yes)
+			)
+		)
+		(property "Description" "Power symbol creates a global label with name \"+3.3V\""
+			(at 325.12 52.07 0)
+			(effects
+				(font
+					(size 1.27 1.27)
+				)
+				(hide yes)
+			)
+		)
+		(pin "1"
+		)
+		(instances
+			(project "uq_phone"
+				(path "/14f57415-6807-40a5-bb38-3cb818a2cdae/3e1644a6-29e0-4613-bdce-8513434c26aa"
+					(reference "#PWR0208")
+					(unit 1)
+				)
+			)
+		)
+	)
+	(symbol
 		(lib_id "power:GND")
 		(at 295.91 124.46 0)
@@
 	)
 	(symbol
-		(lib_id "power:+3.3V")
-		(at 325.12 52.07 0)
+		(lib_id "Misc:MTQH201208S4R7MBT")
+		(at 355.6 41.91 0)
 		(unit 1)
 		(exclude_from_sim no)
@@
 		(on_board yes)
 		(dnp no)
-		(fields_autoplaced yes)
-		(property "Reference" "#PWR069"
-			(at 325.12 55.88 0)
+		(property "Reference" "L2"
+			(at 355.6 37.084 0)
+			(effects
+				(font
+					(size 1.27 1.27)
+				)
+			)
+		)
+		(property "Value" "4.7uH"
+			(at 355.6 39.624 0)
+			(effects
+				(font
+					(size 1.27 1.27)
+				)
+			)
+		)
+		(property "Footprint" "custom_footprints:IND-SMD_L2.0-W1.2_MTQH201208S4R7MBT"
+			(at 355.6 41.91 0)
 			(effects
 				(font
@@
 			)
 		)
-		(property "Value" "+3.3V"
-			(at 325.12 46.99 0)
+		(property "Datasheet" "https://atta.szlcsc.com/upload/public/pdf/source/20230907/B6BF387D97E908951C348B93C86B14B9.pdf"
+			(at 355.6 41.91 0)
 			(effects
 				(font
 					(size 1.27 1.27)
 				)
+				(hide yes)
 			)
 		)
-		(property "Footprint" ""
-			(at 325.12 52.07 0)
+		(property "Description" "Inductance:4.7uH Tolerance:±20% Tolerance:±20% Current - Saturation(Isat):1.6A DC Resistance(DCR):285mΩ"
+			(at 355.6 41.91 0)
 			(effects
 				(font
@@
 			)
 		)
-		(property "Datasheet" ""
-			(at 325.12 52.07 0)
+		(property "Manufacturer Part" "MTQH201208S4R7MBT"
+			(at 355.6 41.91 0)
 			(effects
 				(font
@@
 			)
 		)
-		(property "Description" "Power symbol creates a global label with name \"+3.3V\""
-			(at 325.12 52.07 0)
+		(property "Manufacturer" "MetalLions(美铼)"
+			(at 355.6 41.91 0)
+			(effects
+				(font
+					(size 1.27 1.27)
+				)
+				(hide yes)
+			)
+		)
+		(property "Supplier Part" "C17701166"
+			(at 355.6 41.91 0)
+			(effects
+				(font
+					(size 1.27 1.27)
+				)
+				(hide yes)
+			)
+		)
+		(property "Supplier" "LCSC"
+			(at 355.6 41.91 0)
+			(effects
+				(font
+					(size 1.27 1.27)
+				)
+				(hide yes)
+			)
+		)
+		(property "LCSC Part Name" "4.7uH ±20% 1.6A 温升电流：1.7A"
+			(at 355.6 41.91 0)
 			(effects
 				(font
@@
 		(pin "1"
 		)
+		(pin "2"
+		)
 		(instances
-			(project "uq_phone"
+			(project ""
 				(path "/14f57415-6807-40a5-bb38-3cb818a2cdae/3e1644a6-29e0-4613-bdce-8513434c26aa"
-					(reference "#PWR069")
+					(reference "L2")
 					(unit 1)
 				)

Commit message: Minor Changes - new display
Parts:
- removed Disp1: AFR240320A0-2.0INTM, custom_footprints:Display, symbol Misc:Display
- added DISP1: HS20HS072RX, symbol Misc:HS20HS072RX
Connections:
- net +3.3V: now also DISP1.8 (IOVCC), DISP1.9 (VCC)
- net DISP_CS: now also DISP1.2 (CS)
- net DISP_DC: now also DISP1.3 (RS)
- net DISP_LEDA: now also DISP1.10 (LEDA)
- net DISP_LEDK: now also DISP1.11 (LEDK)
- net GND: now also DISP1.1 (GND), DISP1.12 (GND)
- net uSD_SIM_CD: now also U10.12 (CH5_OUT)
- new net DISP_RESET: DISP1.6 (RESET)
- new net DISP_SCL: DISP1.4 (SCL)
- new net DISP_SDA: DISP1.5 (SDA)
Other:
- note added: "Maybe Change this"
- moved on the sheet: C29, C34, C35, M1, U10, U11, U12

Commit message: New Layout
Parts:
- C27, C28, D2, L2, R29, U9: now not fitted
- DISP1: footprint (none) -> custom_footprints:Display

Commit message: Update layout and BL control
Parts:
- removed C27: 10uF, Capacitor_SMD:C_0603_1608Metric, symbol Capacitors:Capacitor_10uF
- removed C28: 4.7uF, Capacitor_SMD:C_0201_0603Metric, symbol Capacitors:Capacitor_4.7uF
- removed D2: PMEG2010EA, Diode_SMD:D_SOD-323, symbol Misc:PMEG2010EA
- removed L2: 4.7uH, custom_footprints:IND-SMD_L2.0-W1.2_MTQH201208S4R7MBT, symbol Misc:MTQH201208S4R7MBT
- removed R29: 3.83R, Resistor_SMD:R_0402_1005Metric, symbol Resistors:Resistor_3.83R
- removed U9: MCP1664T-E/OT, MCP1664T_E_OT:SOT-23-5_OT_MCH, symbol 2025-04-08_10-28-15:MCP1664T-E_OT
- added Q3: S8050, Package_TO_SOT_SMD:SOT-23, symbol Misc:S8050
- added R21: 10k, Resistor_SMD:R_0201_0603Metric, symbol Resistors:Resistor_10k
- added R26: 1k, Resistor_SMD:R_0402_1005Metric, symbol Resistors:Resistor_1k
- added R27: 10R, Resistor_SMD:R_0402_1005Metric, symbol Resistors:Resistor_10R
Connections:
- net DISP_LEDA is gone; now on net +3.3V_SW: DISP1.10 (LEDA)
- net +3.3V_SW: now also R21.2
- net DISP_BL: now also R26.2
- net DISP_LEDK: now also R27.2
- net GND: now also Q3.2
- new net: Q3.1, R21.1, R26.1
- new net: Q3.3, R27.1
- no-connect marks 13 -> 14
Other:
- note added: "Double Check"
- note removed: "Iout = 0.3/R 3.83R -> 78mA"
- note removed: "Maybe Change this"

Commit message: Several Hours of Routing
Parts:
- removed R27: 10R, Resistor_SMD:R_0402_1005Metric, symbol Resistors:Resistor_10R
- added R27: 5R, Resistor_SMD:R_0402_1005Metric, symbol Resistors:Resistor_5R
Connections:
- net DISP_LEDK: now also R27.2
- net at Q3.3: now also R27.1
Changed lines of the file:
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@@
+	)
+	(symbol
+		(lib_id "Resistors:Resistor_5R")
+		(at 353.06 44.45 0)
+		(unit 1)
+		(exclude_from_sim no)
+		(in_bom yes)
+		(on_board yes)
+		(dnp no)
+		(fields_autoplaced yes)
+		(property "Reference" "R27"
+			(at 355.6 43.1799 0)
+			(effects
+				(font
+					(size 1.27 1.27)
+				)
+				(justify left)
+			)
+		)
+		(property "Value" "5R"
+			(at 355.6 45.7199 0)
+			(effects
+				(font
+					(size 1.27 1.27)
+				)
+				(justify left)
+			)
+		)
+		(property "Footprint" "Resistor_SMD:R_0402_1005Metric"
+			(at 353.06 48.26 0)
+			(effects
+				(font
+					(size 1.27 1.27)
+				)
+				(hide yes)
+			)
+		)
+		(property "Datasheet" ""
+			(at 353.06 48.26 0)
+			(effects
+				(font
+					(size 1.27 1.27)
+				)
+				(hide yes)
+			)
+		)
+		(property "Description" "62.5mW Thick Film Resistor 50V ±1% ±400ppm/℃ 5.1Ω 0402 Chip Resistor - Surface Mount ROHS"
+			(at 353.06 48.26 0)
+			(effects
+				(font
+					(size 1.27 1.27)
+				)
+				(hide yes)
+			)
+		)
+		(property "LCSC PN" "C25128"
+			(at 353.06 44.45 0)
+			(effects
+				(font
+					(size 1.27 1.27)
+				)
+				(hide yes)
+			)
+		)
+		(pin "2"
+		)
+		(pin "1"
+		)
+		(instances
+			(project ""
+				(path "/14f57415-6807-40a5-bb38-3cb818a2cdae/3e1644a6-29e0-4613-bdce-8513434c26aa"
+					(reference "R27")
+					(unit 1)
+				)
+			)
+		)
 	)
 	(symbol
@@
 					(unit 1)
 				)
-			)
-		)
-	)
-	(symbol
-		(lib_id "Resistors:Resistor_10R")
-		(at 353.06 44.45 0)
-		(unit 1)
-		(exclude_from_sim no)
-		(in_bom yes)
-		(on_board yes)
-		(dnp no)
-		(fields_autoplaced yes)
-		(property "Reference" "R27"
-			(at 355.6 43.1799 0)
-			(effects
-				(font
-					(size 1.27 1.27)
-				)
-				(justify left)
-			)
-		)
-		(property "Value" "10R"
-			(at 355.6 45.7199 0)
-			(effects
-				(font
-					(size 1.27 1.27)
-				)
-				(justify left)
-			)
-		)
-		(property "Footprint" "Resistor_SMD:R_0402_1005Metric"
-			(at 353.06 48.26 0)
-			(effects
-				(font
-					(size 1.27 1.27)
-				)
-				(hide yes)
-			)
-		)
-		(property "Datasheet" ""
-			(at 353.06 48.26 0)
-			(effects
-				(font
-					(size 1.27 1.27)
-				)
-				(hide yes)
-			)
-		)
-		(property "Description" "100mW Thick Film Resistor ±100ppm/℃ ±1% 10Ω 0402 Chip Resistor - Surface Mount ROHS"
-			(at 353.06 48.26 0)
-			(effects
-				(font
-					(size 1.27 1.27)
-				)
-				(hide yes)
-			)
-		)
-		(property "LCSC PN" "C413044"
-			(at 353.06 44.45 0)
-			(effects
-				(font
-					(size 1.27 1.27)
-				)
-				(hide yes)
-			)
-		)
-		(pin "2"
-		)
-		(pin "1"
-		)
-		(instances
-			(project ""
-				(path "/14f57415-6807-40a5-bb38-3cb818a2cdae/3e1644a6-29e0-4613-bdce-8513434c26aa"
-					(reference "R27")
-					(unit 1)
-				)

Commit message: Restructure, route and add flex pcb
Parts:
- M1: now left out of the parts list
Changed lines of the file:
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@@
 		(unit 1)
 		(exclude_from_sim no)
-		(in_bom yes)
+		(in_bom no)
 		(on_board yes)
 		(dnp no)
