File: uq_phone_v0.2.0/user_io.kicad_sch (KiCad schematic)
At the start: 17 parts, among them J8 MCS-302S-C1, M1 C08-00A, Q3 S8050, U10 TPD8F003DQDR, U11 LSM6DSVTR, U12 DRV2603RUNR, U8 TPD3F303DQDR

Commit message: Fixed display pinout
Parts:
- DISP1: now left out of the parts list
Other:
- note removed: "Double Check"
- note removed: "TODO: Confirm Switch"
- moved on the sheet: C34, C35, DISP1, Q3, R21, R26, R27, U11

Commit message: Cleaning up adn fixing massive mistake
Other:
- note added: "UQ Phone"
- note removed: "Backlight Driver"
- note removed: "Display"
- note removed: "IMU"
- note removed: "Micro SD Card"
- note removed: "Micro SIM card"
- note removed: "Motor & Vibration"
- title: UQ Phone -> I/O  System
- moved on the sheet: C29, C32, C33, C34, C35, DISP1, J8A, J8B, M1, Q3, R21, R25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

Commit message: minor comments
Other:
- note added: "This 3.3v VDD should not be activated until insertion, requires fixing"
Changed lines of the file:
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@@
+		)
+	)
+	(text "This 3.3v VDD should not be activated\nuntil insertion, requires fixing"
+		(exclude_from_sim no)
+		(at 102.108 77.978 0)
+		(effects
+			(font
+				(size 1.27 1.27)
+				(thickness 0.254)
+				(bold yes)
+				(color 255 0 0 1)
+			)
 		)
 	)
