File: uq_phone_v0.2.0/uq_phone.kicad_sch (KiCad schematic)
At the start: 0 parts

Commit message: Various Changes to footprints and components
Other:
- title: (none) -> UQ Phone
Changed lines of the file:
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@@
 	(paper "A3")
 	(title_block
+		(title "UQ Phone")
+		(rev "0.2.0")
 		(company "The University of Queensland")
 	)

Commit message: Cleaning up adn fixing massive mistake
Other:
- note added: "UQ Phone"
Changed lines of the file:
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@@
 	(title_block
 		(title "UQ Phone")
+		(date "2025-09-05")
 		(rev "0.2.0")
 		(company "The University of Queensland")
+		(comment 1 "James Wood")
+	)
+	(text "UQ Phone"
+		(exclude_from_sim no)
+		(at 316.23 258.064 0)
+		(effects
+			(font
+				(size 4 4)
+				(thickness 0.8)
+				(bold yes)
+				(color 132 0 0 1)
+			)
+		)
 	)
 	(sheet
