File: uq_phone_v0.2.0/uq_phone_v0.2.0_cellular/uq_phone_cellular/uq_phone_cellular.kicad_pcb (KiCad board)
At the start: 4 copper layers, 45 x 30.2 mm, 32 parts, among them J1 513382474, J2 513382474, J3 20279-001E-03, J4 20279-001E-03, U1 WP SNAP-IN BASE_6000636

Commit message: More roting and vias
Parts:
- moved J4 0.10 mm to (117.4, 73.8)
Routing:
- net MOB_MAIN_ANT: track 0.00 -> 7.05 mm
- net MOB_AUX_ANT: track 0.00 -> 6.17 mm

Commit message: DRC and routing fixing
Parts:
- moved TP7 5.43 mm to (122.2, 65.5)
- moved TP10 5.38 mm to (116.5, 68.4)
- moved TP6 4.96 mm to (119.1, 65.8)
- moved TP9 3.44 mm to (119.0, 68.4)
- moved TP8 2.87 mm to (122.1, 68.2)
- moved TP5 1.79 mm to (116.5, 65.8)
- moved TP4 1.74 mm to (116.5, 63.2)
Routing:
- net Net-(U1A-J4): track 0.67 -> 39.1 mm, vias 1 -> 2
- net Net-(U1A-J5): track 0.67 -> 38.0 mm, vias 1 -> 2
- net Net-(U1A-J3): track 0.67 -> 36.7 mm, vias 1 -> 2
- net Net-(U1A-J1): track 0.67 -> 36.5 mm, vias 1 -> 2
- net Net-(U1A-J2): track 0.67 -> 34.8 mm, vias 1 -> 2
- net Net-(U1A-J6): track 0.67 -> 34.1 mm, vias 1 -> 2
- net Net-(U1A-J7): track 0.67 -> 30.6 mm, vias 1 -> 2
- net Net-(U1A-TX_ON): track 0.00 -> 18.7 mm, vias 0 -> 2
- net MOB_PWR: track 37.8 -> 43.5 mm
- net MOB_RST: track 20.4 -> 24.9 mm
- net MOB_SAFE_PWR_REMOVE_L: track 40.0 -> 43.8 mm
- net GND: track 7.01 -> 8.01 mm, vias 268 -> 300
