File: uq_phone_v0.1.0/uq_phone_v0.1.0_io_board/front_board.kicad_sch (KiCad schematic)
At the start: 61 parts, among them J1 6871XX14022_68715014022, J9 541324562, SW1 SKTAAAE010, SW10 SKTAAAE010, SW11 SKTAAAE010, SW12 SKTAAAE010, SW13 SKTAAAE010, SW14 SKTAAAE010, SW15 SKTAAAE010, SW16 SKTAAAE010, SW17 SKTAAAE010, SW18 SKTAAAE010, SW19 SKTAAAE010, SW2 SKTAAAE010, SW20 SKTAAAE010, SW21 SKTAAAE010, SW22 SKTAAAE010, SW23 SKTAAAE010, SW24 SKTAAAE010, SW25 SKTAAAE010, SW27 SKTAAAE010, SW29 SKTAAAE010, SW3 SKTAAAE010, SW31 SKTAAAE010, SW33 SKTAAAE010, SW34 SKTAAAE010, SW35 SKTAAAE010, SW36 SKTAAAE010, SW37 SKTAAAE010, SW38 SKTAAAE010, SW39 SKTAAAE010, SW4 SKTAAAE010, SW40 SKTAAAE010, SW41 SKTAAAE010, SW42 SKTAAAE010, SW43 SKSCLCE010, SW44 SKSCLCE010, SW45 SKSCLCE010, SW5 SKTAAAE010, SW6 SKTAAAE010, SW7 SKTAAAE010, SW8 SKTAAAE010, SW9 SKTAAAE010

Commit message: Cleaning up adn fixing massive mistake
Other:
- title: (none) -> IO Board
Changed lines of the file:
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@@
 	(generator_version "9.0")
 	(paper "A3")
+	(title_block
+		(title "IO Board")
+	)
 	(text "D-Pad Buttons\n"
 		(exclude_from_sim no)
